File: hardware/pcb/kveld_rev_a/kveld_rev_a.kicad_pcb (KiCad board)
At the start: 4 copper layers, 78 x 45 mm, 0 parts

Commit message: docs(hw): improve rev a render resolution
Other:
- board text added: "ANTENNA — NO COPPER / METAL"
- board text added: "CONSTRAINT SKELETON — NOT FOR FABRICATION"
- board text added: "WROOM-1 CONFLICT / 1U BASELINE"
- board text removed: "NO COPPER / NO METAL — MODULE ANTENNA"
- board text removed: "REV A CONSTRAINT SKELETON — NOT FOR FABRICATION"
- board text removed: "WROOM-1 CONFLICT STUDY / 1U BASELINE"
Changed lines of the file:
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@@
 	(gr_circle (center 6.5 28) (end 7.75 28) (stroke (width 0.15) (type dash)) (fill no) (layer "User.1"))
 	(gr_circle (center 77.5 28) (end 78.75 28) (stroke (width 0.15) (type dash)) (fill no) (layer "User.1"))
-	(gr_text "REV A CONSTRAINT SKELETON — NOT FOR FABRICATION" (at 42 38 0) (layer "Cmts.User") (effects (font (size 1.2 1.2) (thickness 0.18))))
+	(gr_text "CONSTRAINT SKELETON — NOT FOR FABRICATION" (at 48 28 0) (layer "Cmts.User") (effects (font (size 0.75 0.75) (thickness 0.12))))
 	(gr_text "CELL 503035 KEEP-OUT" (at 42 19 0) (layer "User.2") (effects (font (size 1 1) (thickness 0.15))))
-	(gr_text "NO COPPER / NO METAL — MODULE ANTENNA" (at 9 28 90) (layer "User.2") (effects (font (size 0.8 0.8) (thickness 0.12))))
+	(gr_text "ANTENNA — NO COPPER / METAL" (at 9 28 90) (layer "User.2") (effects (font (size 0.65 0.65) (thickness 0.1))))
 	(gr_text "DISPLAY ENVELOPE ABOVE" (at 42 35 0) (layer "User.1") (effects (font (size 1 1) (thickness 0.15))))
 	(gr_text "USB-C" (at 42 46 0) (layer "F.SilkS") (effects (font (size 0.8 0.8) (thickness 0.12))))
 	(gr_text "KVELD REV A0" (at 69 5.5 0) (layer "F.SilkS") (effects (font (size 1 1) (thickness 0.15))))
 	(gr_text "FPC DATUM — VERIFY FOOTPRINT" (at 42 40 0) (layer "User.1") (effects (font (size 0.65 0.65) (thickness 0.1))))
-	(gr_text "WROOM-1 CONFLICT STUDY / 1U BASELINE" (at 16 28 90) (layer "Cmts.User") (effects (font (size 0.65 0.65) (thickness 0.1))))
+	(gr_text "WROOM-1 CONFLICT / 1U BASELINE" (at 16 28 90) (layer "Cmts.User") (effects (font (size 0.55 0.55) (thickness 0.09))))
 	(zone
 		(net 0)
