File: hardware/pcb/kveld_rev_a/kveld_rev_a.kicad_sch (KiCad schematic)
At the start: 0 parts

Commit message: feat(hw): capture rev a schematic and refine enclosure
Other:
- sheet 3V3 regulation renamed 3V3 buck-boost regulation

Commit message: refactor(hw): consolidate and clarify schematic
Other:
- sheet Battery charger renamed Power and USB
- sheet E-paper interface renamed E-paper display
- sheet ESP32-S3 core renamed Controller and user I/O
- removed sheet 3V3 buck-boost regulation
- removed sheet Controls and status
- removed sheet Programming and test
- removed sheet USB and protection
- title: (none) -> Kveld Rev A schematic overview
Changed lines of the file:
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@@
 	(generator_version "10.0")
 	(paper "A4")
+	(title_block (title "Kveld Rev A schematic overview") (rev "Rev A"))
 	(sheet
-		(at 157.48 25.4)
+		(at 25.4 45.72)
 		(size 50.8 25.4)
 		(exclude_from_sim no)
@@
 			(color 0 0 0 0)
 		)
-		(property "Sheetname" "3V3 buck-boost regulation"
-			(at 157.48 24.6884 0)
+		(property "Sheetname" "Power and USB"
+			(at 25.4 45.0084 0)
 			(show_name no)
 			(do_not_autoplace no)
@@
 			)
 		)
-		(property "Sheetfile" "sheets/regulator.kicad_sch"
-			(at 157.48 51.5116 0)
+		(property "Sheetfile" "sheets/battery_charger.kicad_sch"
+			(at 25.4 71.8316 0)
 			(show_name no)
 			(do_not_autoplace no)
@@
 			(project "kveld_rev_a"
 				(path "/9b5e4c31-c66f-4b64-9ff8-62a2c447d0bc"
-					(page "7")
+					(page "2")
 				)
 			)
 		)
 	)
-	(sheet
-		(at 91.44 111.76)
+(sheet
+		(at 104.14 45.72)
 		(size 50.8 25.4)
 		(exclude_from_sim no)
@@
 			(color 0 0 0 0)
 		)
-		(property "Sheetname" "Programming and test"
-			(at 91.44 111.0484 0)
-			(show_name no)
-			(do_not_autoplace no)
-			(effects
-				(font
-					(size 1.27 1.27)
-				)
-				(justify left bottom)
-			)
-		)
-		(property "Sheetfile" "sheets/programming_test.kicad_sch"
-			(at 91.44 137.8716 0)
-			(show_name no)
-			(do_not_autoplace no)
-			(effects
-				(font
-					(size 1.27 1.27)
-				)
-				(justify left top)
-			)
-		)
-		(instances
-			(project "kveld_rev_a"
-				(path "/9b5e4c31-c66f-4b64-9ff8-62a2c447d0bc"
-					(page "6")
-				)
-			)
-		)
-	)
-	(sheet
-		(at 157.48 68.58)
-		(size 50.8 25.4)
-		(exclude_from_sim no)
-		(in_bom yes)
-		(on_board yes)
-		(dnp no)
-		(fields_autoplaced yes)
-		(stroke
-			(width 0)
-			(type solid)
-		)
-		(fill
-			(color 0 0 0 0)
-		)
-		(property "Sheetname" "Controls and status"
-			(at 157.48 67.8684 0)
-			(show_name no)
-			(do_not_autoplace no)
-			(effects
-				(font
-					(size 1.27 1.27)
-				)
-				(justify left bottom)
-			)
-		)
-		(property "Sheetfile" "sheets/controls_status.kicad_sch"
-			(at 157.48 94.6916 0)
-			(show_name no)
-			(do_not_autoplace no)
-			(effects
-				(font
-					(size 1.27 1.27)
-				)
-				(justify left top)
-			)
-		)
-		(instances
-			(project "kveld_rev_a"
-				(path "/9b5e4c31-c66f-4b64-9ff8-62a2c447d0bc"
-					(page "8")
-				)
-			)
-		)
-	)
-	(sheet
-		(at 25.4 68.58)
-		(size 50.8 25.4)
-		(exclude_from_sim no)
-		(in_bom yes)
-		(on_board yes)
-		(dnp no)
-		(fields_autoplaced yes)
-		(stroke
-			(width 0)
-			(type solid)
-		)
-		(fill
-			(color 0 0 0 0)
-		)
-		(property "Sheetname" "ESP32-S3 core"
-			(at 25.4 67.8684 0)
+		(property "Sheetname" "Controller and user I/O"
+			(at 104.14 45.0084 0)
 			(show_name no)
 			(do_not_autoplace no)
@@
 		)
 		(property "Sheetfile" "sheets/esp32_core.kicad_sch"
-			(at 25.4 94.6916 0)
+			(at 104.14 71.8316 0)
 			(show_name no)
 			(do_not_autoplace no)
@@
 		)
 	)
-	(sheet
-		(at 91.44 25.4)
+(sheet
+		(at 182.88 45.72)
 		(size 50.8 25.4)
 		(exclude_from_sim no)
@@
 			(color 0 0 0 0)
 		)
-		(property "Sheetname" "Battery charger"
-			(at 91.44 24.6884 0)
+		(property "Sheetname" "E-paper display"
+			(at 182.88 45.0084 0)
 			(show_name no)
 			(do_not_autoplace no)
@@
 			)
 		)
-		(property "Sheetfile" "sheets/battery_charger.kicad_sch"
-			(at 91.44 51.5116 0)
+		(property "Sheetfile" "sheets/epaper.kicad_sch"
+			(at 182.88 71.8316 0)
 			(show_name no)
 			(do_not_autoplace no)
@@
 				)
 			)
-		)
-	)
-	(sheet
-		(at 91.44 68.58)
-		(size 50.8 25.4)
-		(exclude_from_sim no)
-		(in_bom yes)
-		(on_board yes)
-		(dnp no)
-		(fields_autoplaced yes)
-		(stroke
-			(width 0)
-			(type solid)
-		)
-		(fill
-			(color 0 0 0 0)
-		)
-		(property "Sheetname" "E-paper interface"
-			(at 91.44 67.8684 0)
-			(show_name no)
-			(do_not_autoplace no)
-			(effects
-				(font
-					(size 1.27 1.27)
-				)
-				(justify left bottom)
-			)
-		)
-		(property "Sheetfile" "sheets/epaper.kicad_sch"
-			(at 91.44 94.6916 0)
-			(show_name no)
-			(do_not_autoplace no)
-			(effects
-				(font
-					(size 1.27 1.27)
-				)
-				(justify left top)
-			)
-		)
-		(instances
-			(project "kveld_rev_a"
-				(path "/9b5e4c31-c66f-4b64-9ff8-62a2c447d0bc"
-					(page "5")
-				)
-			)
-		)
-	)
-	(sheet
-		(at 25.4 25.4)
-		(size 50.8 25.4)
-		(exclude_from_sim no)
-		(in_bom yes)
-		(on_board yes)
-		(dnp no)
-		(fields_autoplaced yes)
-		(stroke
-			(width 0)
-			(type solid)
-		)
-		(fill
-			(color 0 0 0 0)
-		)
-		(property "Sheetname" "USB and protection"
-			(at 25.4 24.6884 0)
-			(show_name no)
-			(do_not_autoplace no)
-			(effects
-				(font
-					(size 1.27 1.27)
-				)
-				(justify left bottom)
-			)
-		)
-		(property "Sheetfile" "sheets/usb_protection.kicad_sch"
-			(at 25.4 51.5116 0)
-			(show_name no)
-			(do_not_autoplace no)
-			(effects
-				(font
-					(size 1.27 1.27)
-				)
-				(justify left top)
-			)
-		)
-		(instances
-			(project "kveld_rev_a"
-				(path "/9b5e4c31-c66f-4b64-9ff8-62a2c447d0bc"
-					(page "2")
-				)
-			)
