File: hardware/pcb/kveld_rev_a/sheets/controls_status.kicad_sch (KiCad schematic)
At the start: 0 parts

Commit message: feat(hw): capture rev a schematic and refine enclosure
Parts:
- added C25, C26: 10nF, Capacitor_SMD:C_0603_1608Metric, symbol Device:C
- added D4: APBA2006SURKCGKC red/green, symbol Device:LED_Dual_AAKK
- added R21, R22: 47k, Resistor_SMD:R_0603_1608Metric, symbol Device:R
- added R23, R24: 1k, Resistor_SMD:R_0603_1608Metric, symbol Device:R
- added SW1: CATEGORY KSC321GLFS, symbol Switch:SW_Push
- added SW2: NEXT KSC321GLFS, symbol Switch:SW_Push
Connections:
- new net 3V3: R21.1, R22.1
- new net BTN_CATEGORY: C25.1, R21.2, SW1.1
- new net BTN_NEXT: C26.1, R22.2, SW2.1
- new net GND: C25.2, C26.2, D4.3 (K1), D4.4 (K2), SW1.2, SW2.2
- new net LED_GREEN_A: D4.2 (A2), R24.2
- new net LED_RED_A: D4.1 (A1), R23.2
- new net STATUS_GREEN: R24.1
- new net STATUS_RED: R23.1
Other:
- note added: "External pull-ups preserve RTC wake behaviour. LED dies are driven active-high through 1 kΩ."
- title: (none) -> Buttons and red/green status LED
