File: hardware/pcb/kveld_rev_a/sheets/programming_test.kicad_sch (KiCad schematic)
At the start: 0 parts

Commit message: feat(hw): capture rev a schematic and refine enclosure
Parts:
- added J4: TC2030 recovery pads, Connector:Tag-Connect_TC2030-IDC-NL_2x03_P1.27mm_Vertical, symbol Connector_Generic:Conn_02x03_Odd_Even
- added TP1: BOOT_IO0, TestPoint:TestPoint_Pad_D1.0mm, symbol Connector:TestPoint
- added TP10: USB_VBUS, TestPoint:TestPoint_Pad_D1.0mm, symbol Connector:TestPoint
- added TP11: REG_PG, TestPoint:TestPoint_Pad_D1.0mm, symbol Connector:TestPoint
- added TP2: CHIP_EN, TestPoint:TestPoint_Pad_D1.0mm, symbol Connector:TestPoint
- added TP3: GND, TestPoint:TestPoint_Pad_D1.0mm, symbol Connector:TestPoint
- added TP4: UART0_TX, TestPoint:TestPoint_Pad_D1.0mm, symbol Connector:TestPoint
- added TP5: UART0_RX, TestPoint:TestPoint_Pad_D1.0mm, symbol Connector:TestPoint
- added TP6: FACTORY_RESET_OD, TestPoint:TestPoint_Pad_D1.0mm, symbol Connector:TestPoint
- added TP7: 3V3, TestPoint:TestPoint_Pad_D1.0mm, symbol Connector:TestPoint
- added TP8: VBAT, TestPoint:TestPoint_Pad_D1.0mm, symbol Connector:TestPoint
- added TP9: VSYS, TestPoint:TestPoint_Pad_D1.0mm, symbol Connector:TestPoint
Connections:
- new net 3V3: J4.1 (Pin_1), TP7.1
- new net BOOT_IO0: J4.4 (Pin_4), TP1.1
- new net CHIP_EN: J4.3 (Pin_3), TP2.1
- new net FACTORY_RESET_OD: TP6.1
- new net GND: J4.2 (Pin_2), TP3.1
- new net REG_PG: TP11.1
- new net UART0_RX: J4.6 (Pin_6), TP5.1
- new net UART0_TX: J4.5 (Pin_5), TP4.1
- new net USB_VBUS: TP10.1
- new net VBAT: TP8.1
- new net VSYS: TP9.1
Other:
- note added: "USB is the normal flash/serial/debug path. The underside Tag-Connect pads recover IO0, EN, and UART0."
- title: (none) -> Recovery and production test access
