File: hardware/pcb/kveld_rev_a/sheets/regulator.kicad_sch (KiCad schematic)
At the start: 0 parts

Commit message: feat(hw): capture rev a schematic and refine enclosure
Parts:
- added C10: 47uF 6.3V, Capacitor_SMD:C_0805_2012Metric, symbol Device:C
- added C11: 100nF, Capacitor_SMD:C_0603_1608Metric, symbol Device:C
- added C8: 10uF 6.3V, Capacitor_SMD:C_0603_1608Metric, symbol Device:C
- added C9: 22uF 6.3V, Capacitor_SMD:C_0603_1608Metric, symbol Device:C
- added L2: 0.47uH XFL4015-471ME, symbol Device:L
- added R14: 511k 1%, Resistor_SMD:R_0603_1608Metric, symbol Device:R
- added R15: 91k 1%, Resistor_SMD:R_0603_1608Metric, symbol Device:R
- added R16: 100k, Resistor_SMD:R_0603_1608Metric, symbol Device:R
- added U3: TPS63802DLA, symbol Kveld:TPS63802DLA
Connections:
- new net 3V3: C10.1, C11.1, C9.1, R14.1, R16.1, U3.6 (VOUT)
- new net GND: C10.2, C11.2, C8.2, C9.2, R15.2, U3.2 (MODE), U3.3 (AGND), U3.8 (GND)
- new net REG_FB: R14.2, R15.1, U3.4 (FB)
- new net REG_L1: L2.1, U3.9 (L1)
- new net REG_L2: L2.2, U3.7 (L2)
- new net REG_PG: R16.2, U3.5 (PG)
- new net VSYS: C8.1, U3.1 (EN), U3.10 (VIN)
Other:
- note added: "TPS63802 keeps 3.3 V regulated over the protected LiPo discharge range; MODE is low for PFM."
- title: (none) -> 3.3 V low-IQ buck-boost regulator
