File: hardware/pcb/kveld_rev_a/sheets/usb_protection.kicad_sch (KiCad schematic)
At the start: 0 parts

Commit message: feat(hw): capture rev a schematic and refine enclosure
Parts:
- added C1, C2: 3pF DNP, Capacitor_SMD:C_0603_1608Metric, symbol Device:C
- added C3: 100nF, Capacitor_SMD:C_0603_1608Metric, symbol Device:C
- added J1: USB-C receptacle, Connector_USB:USB_C_Receptacle_HRO_TYPE-C-31-M-12, symbol Connector:USB_C_Receptacle_USB2.0_16P
- added R1, R2: 5.1k, Resistor_SMD:R_0603_1608Metric, symbol Device:R
- added R3, R4: 22, Resistor_SMD:R_0603_1608Metric, symbol Device:R
- added R5: 150k, Resistor_SMD:R_0603_1608Metric, symbol Device:R
- added R6: 100k, Resistor_SMD:R_0603_1608Metric, symbol Device:R
- added U4: USBLC6-2SC6, Package_TO_SOT_SMD:SOT-23-6, symbol Kveld:USBLC6-2SC6
Connections:
- new net GND: C1.2, C2.2, C3.2, J1.A1 (GND), J1.A12 (GND), J1.B1 (GND), J1.B12 (GND), R1.2, R2.2, R6.2, U4.2 (GND)
- new net USB_CC1: J1.A5 (CC1), R1.1
- new net USB_CC2: J1.B5 (CC2), R2.1
- new net USB_DN: C2.1, R4.2
- new net USB_DN_CONN: J1.A7 (D-), J1.B7 (D-), U4.3 (I/O2)
- new net USB_DN_ESD: R4.1, U4.4 (I/O2)
- new net USB_DP: C1.1, R3.2
- new net USB_DP_CONN: J1.A6 (D+), J1.B6 (D+), U4.1 (I/O1)
- new net USB_DP_ESD: R3.1, U4.6 (I/O1)
- new net USB_VBUS: J1.A4 (VBUS), J1.A9 (VBUS), J1.B4 (VBUS), J1.B9 (VBUS), R5.1, U4.5 (VBUS)
- new net VBUS_SENSE: C3.1, R5.2, R6.1
- no-connect marks 0 -> 3
Other:
- note added: "One USB-C port supplies 5 V and provides ESP32-S3 USB Serial/JTAG. No USB-PD."
- title: (none) -> USB-C and native USB protection
