File: hardware/pcb/kveld_rev_a/sheets/battery_charger.kicad_sch (KiCad schematic)
At the start: 34 parts, among them J1 USB-C receptacle, J3 Protected LiPo + NTC, U2 BQ25185DLH, U3 TPS63802DLA, U4 USBLC6-2SC6, U5 TPS22917DBVR

Commit message: fix(hw): correct rev A charger/regulator wiring and assign footprints
Two schematic errors that ERC could not catch, both electrically valid
but topologically wrong:

- TPS63802 feedback divider was shorted: a straight wire tied FB to VOUT
  and bypassed R14, so the part would regulate the 3.3 V rail down to its
  0.5 V reference. Rewired VOUT -> R14 -> FB node -> R15 -> GND (3.31 V).
- BQ25185 TS/MR and the pack NTC wire (J3.2) were tied to VBAT, which the
  charger reads as an out-of-range temperature and suspends charging.
  TS/MR is now the BATT_NTC net carrying only J3.2; BAT stays on VBAT.
  The 38 uA TS source and the 10 kOhm B=3435 pack NTC to GND need no
  external bias (~1.5 C / ~59 C window).

Footprints: every symbol now carries one. SW1/SW2 use the KiCad
CK_KSC6xxG land (matches the KSC3 drawing). Four parts with no library
match get project land patterns in kveld.pretty (registered via
fp-lib-table): Texas_DLA0010A_VSON-HR-10 (no exposed pad), L_Coilcraft_
XFL4015, L_TDK_VLS4012, and a preliminary LED_Kingbright_APBA2006 whose
pad numbers follow the LED_Dual_AAKK symbol.

Also regroup TP1-TP11 from a full-width row into a compact two-row block,
and ignore the KiCad Local-History plugin's nested git repo.

ERC, constraint-board DRC, BOM and STEP export still pass.

Co-Authored-By: Claude Opus 4.8 <noreply@anthropic.com>
Parts:
- L2: footprint (none) -> kveld:L_Coilcraft_XFL4015
- U3: footprint (none) -> kveld:Texas_DLA0010A_VSON-HR-10_2x3mm_P0.5mm
Connections:
- net 3V3: no longer R14.2, R15.1, U3.4 (FB)
- net VBAT: no longer J3.2 (Pin_2), U2.6 (TS/MR)
- new net: R14.2, R15.1, U3.4 (FB)
- new net BATT_NTC: J3.2 (Pin_2), U2.6 (TS/MR)
Changed lines of the file:
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@@
-	)
-	(junction
-		(at 66.04 137.16)
-		(diameter 0)
-		(color 0 0 0 0)
-	)
-	(junction
-		(at 86.36 137.16)
-		(diameter 0)
-		(color 0 0 0 0)
 	)
 	(junction
@@
 	)
 	(junction
-		(at 248.92 87.63)
-		(diameter 0)
-		(color 0 0 0 0)
-	)
-	(junction
-		(at 248.92 95.25)
-		(diameter 0)
-		(color 0 0 0 0)
-	)
-	(junction
 		(at 60.96 58.42)
 		(diameter 0)
@@
 	)
 	(junction
-		(at 104.14 137.16)
-		(diameter 0)
-		(color 0 0 0 0)
-	)
-	(junction
 		(at 185.42 102.87)
 		(diameter 0)
@@
 	)
 	(junction
-		(at 63.5 137.16)
-		(diameter 0)
-		(color 0 0 0 0)
-	)
-	(junction
 		(at 185.42 100.33)
 		(diameter 0)
@@
 	(wire
 		(pts
-			(xy 241.3 63.5) (xy 248.92 63.5)
-		)
-		(stroke
-			(width 0)
-			(type default)
-		)
-	)
-	(wire
-		(pts
 			(xy 271.78 152.4) (xy 271.78 153.67)
 		)
@@
 	(wire
 		(pts
+			(xy 241.3 63.5) (xy 246.38 63.5)
+		)
+		(stroke
+			(width 0)
+			(type default)
+		)
+	)
+	(wire
+		(pts
+			(xy 246.38 63.5) (xy 246.38 101.6)
+		)
+		(stroke
+			(width 0)
+			(type default)
+		)
+	)
+	(wire
+		(pts
+			(xy 246.38 101.6) (xy 248.92 101.6)
+		)
+		(stroke
+			(width 0)
+			(type default)
+		)
+	)
+	(wire
+		(pts
+			(xy 248.92 95.25) (xy 248.92 107.95)
+		)
+		(stroke
+			(width 0)
+			(type default)
+		)
+	)
+	(wire
+		(pts
+			(xy 248.92 85.09) (xy 248.92 87.63)
+		)
+		(stroke
+			(width 0)
+			(type default)
+		)
+	)
+	(junction
+		(at 248.92 101.6)
+		(diameter 0)
+		(color 0 0 0 0)
+	)
+	(wire
+		(pts
 			(xy 139.7 68.58) (xy 139.7 62.23)
 		)
@@
 	(wire
 		(pts
-			(xy 248.92 63.5) (xy 248.92 107.95)
-		)
-		(stroke
-			(width 0)
-			(type default)
-		)
-	)
-	(wire
-		(pts
 			(xy 220.98 58.42) (xy 218.44 58.42)
 		)
@@
 	(wire
 		(pts
-			(xy 63.5 137.16) (xy 104.14 137.16)
-		)
-		(stroke
-			(width 0)
-			(type default)
-		)
-	)
-	(wire
-		(pts
 			(xy 185.42 100.33) (xy 185.42 102.87)
 		)
@@
 			(width 0)
 			(type default)
+		)
+	)
+	(wire
+		(pts
+			(xy 86.36 137.16) (xy 88.9 137.16)
+		)
+		(stroke
+			(width 0)
+			(type default)
+		)
+	)
+	(global_label "BATT_NTC"
+		(shape passive)
+		(at 66.04 137.16 180)
+		(fields_autoplaced yes)
+		(effects
+			(font
+				(size 0.9 0.9)
+			)
+			(justify right)
+		)
+		(property "Intersheetrefs" "${INTERSHEET_REFS}"
+			(at 66.04 137.16 180)
+			(hide yes)
+			(show_name no)
+			(do_not_autoplace no)
+			(effects
+				(font
+					(size 0.8 0.8)
+				)
+			)
+		)
+	)
+	(global_label "BATT_NTC"
+		(shape passive)
+		(at 104.14 137.16 0)
+		(fields_autoplaced yes)
+		(effects
+			(font
+				(size 0.9 0.9)
+			)
+			(justify left)
+		)
+		(property "Intersheetrefs" "${INTERSHEET_REFS}"
+			(at 104.14 137.16 0)
+			(hide yes)
+			(show_name no)
+			(do_not_autoplace no)
+			(effects
+				(font
+					(size 0.8 0.8)
+				)
+			)
 		)
 	)
@@
 			)
 		)
-		(property "Footprint" ""
+		(property "Footprint" "kveld:L_Coilcraft_XFL4015"
 			(at 231.14 35.56 0)
 			(hide yes)
@@
 			)
 		)
-		(property "Footprint" ""
+		(property "Footprint" "kveld:Texas_DLA0010A_VSON-HR-10_2x3mm_P0.5mm"
 			(at 231.14 60.96 0)
 			(hide yes)
