File: hardware/pcb/kveld_rev_a/sheets/epaper.kicad_sch (KiCad schematic)
At the start: 23 parts, among them J2 FH12-24S-0.5SH, Q1 Si1308EDL, U6 TPS22917DBVR

Commit message: fix(hw): correct rev A charger/regulator wiring and assign footprints
Two schematic errors that ERC could not catch, both electrically valid
but topologically wrong:

- TPS63802 feedback divider was shorted: a straight wire tied FB to VOUT
  and bypassed R14, so the part would regulate the 3.3 V rail down to its
  0.5 V reference. Rewired VOUT -> R14 -> FB node -> R15 -> GND (3.31 V).
- BQ25185 TS/MR and the pack NTC wire (J3.2) were tied to VBAT, which the
  charger reads as an out-of-range temperature and suspends charging.
  TS/MR is now the BATT_NTC net carrying only J3.2; BAT stays on VBAT.
  The 38 uA TS source and the 10 kOhm B=3435 pack NTC to GND need no
  external bias (~1.5 C / ~59 C window).

Footprints: every symbol now carries one. SW1/SW2 use the KiCad
CK_KSC6xxG land (matches the KSC3 drawing). Four parts with no library
match get project land patterns in kveld.pretty (registered via
fp-lib-table): Texas_DLA0010A_VSON-HR-10 (no exposed pad), L_Coilcraft_
XFL4015, L_TDK_VLS4012, and a preliminary LED_Kingbright_APBA2006 whose
pad numbers follow the LED_Dual_AAKK symbol.

Also regroup TP1-TP11 from a full-width row into a compact two-row block,
and ignore the KiCad Local-History plugin's nested git repo.

ERC, constraint-board DRC, BOM and STEP export still pass.

Co-Authored-By: Claude Opus 4.8 <noreply@anthropic.com>
Parts:
- L1: footprint (none) -> kveld:L_TDK_VLS4012
Changed lines of the file:
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@@
 			)
 		)
-		(property "Footprint" ""
+		(property "Footprint" "kveld:L_TDK_VLS4012"
 			(at 104.14 50.8 0)
 			(hide yes)
