File: hardware/pcb/cicala_rev_a/cicala_rev_a.kicad_sch (KiCad schematic)
At the start: 0 parts

Commit message: feat: rename project and adopt Cicala identity
Other:
- title: Kveld Rev A schematic overview -> Cicala Rev A schematic overview
Changed lines of the file:
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@@
 	(paper "A4")
 	(title_block
-		(title "Kveld Rev A schematic overview")
+		(title "Cicala Rev A schematic overview")
 		(rev "Rev A")
 	)
@@
 		)
 		(instances
-			(project "kveld_rev_a"
+			(project "cicala_rev_a"
 				(path "/9b5e4c31-c66f-4b64-9ff8-62a2c447d0bc"
 					(page "3")
@@
 		)
 		(instances
-			(project "kveld_rev_a"
+			(project "cicala_rev_a"
 				(path "/9b5e4c31-c66f-4b64-9ff8-62a2c447d0bc"
 					(page "2")
@@
 		)
 		(instances
-			(project "kveld_rev_a"
+			(project "cicala_rev_a"
 				(path "/9b5e4c31-c66f-4b64-9ff8-62a2c447d0bc"
 					(page "4")
