File: hardware/pcb/cicala_rev_a/sheets/battery_charger.kicad_sch (KiCad schematic)
At the start: 34 parts, among them J1 USB-C receptacle, J3 Protected LiPo + NTC, U2 BQ25185DLH, U3 TPS63802DLA, U4 USBLC6-2SC6, U5 TPS22917DBVR

Commit message: feat: rename project and adopt Cicala identity
Parts:
- L2: footprint kveld:L_Coilcraft_XFL4015 -> cicala:L_Coilcraft_XFL4015
- U2: symbol Kveld:BQ25185DLH -> Cicala:BQ25185DLH
- U3: footprint kveld:Texas_DLA0010A_VSON-HR-10_2x3mm_P0.5mm -> cicala:Texas_DLA0010A_VSON-HR-10_2x3mm_P0.5mm; symbol Kveld:TPS63802DLA -> Cicala:TPS63802DLA
- U4: symbol Kveld:USBLC6-2SC6 -> Cicala:USBLC6-2SC6
