File: hardware/pcb/cicala_rev_a/sheets/battery_charger.kicad_sch (KiCad schematic)
At the start: 35 parts, among them J1 USB-C receptacle, J3 Protected LiPo + NTC, U2 BQ25185DLH, U3 TPS63802DLA, U4 USBLC6-2SC6, U5 TPS22917DBVR

Commit message: feat(hw): route the Rev A board, and correct three part ratings
Board work. The layer plan is F.Cu and B.Cu for signals with a ground pour,
In1.Cu as an unbroken ground reference, and In2.Cu carrying the 3V3 plane,
signals, and a ground island under the USB pair so that pair is referenced to
ground rather than to the rail. Two signal layers were not enough for 105
parts on 78 x 49 mm.

Placement and routing are generated by hardware/pcb/tools/ rather than dragged
by hand, so they can be regenerated after a schematic change and read as a
diff. The router is a grid maze router with hard blocking, so clearance is a
property of the search rather than something checked afterwards. Getting that
right took finding five modelling errors, each recorded in tools/README.md;
the one that mattered most is that copper modelled as grid cells can extend
half a cell past the outermost cell centre, so every clearance radius has to
carry that slack. Ignoring it produced violations the model could not see.

The board is not finished: 36 connections are unrouted and about 50 DRC
violations remain, mostly pour artifacts around the unrouted areas. The
READMEs say so rather than implying otherwise.

Part ratings, each against the datasheet rather than by habit:

- C8 becomes 10 uF 25 V in 0805. SLUSF65B section 7.2.2.3 asks for 25 V parts
  on the charger's IN and SYS pins, and the TPS63802 wants 4 uF effective on
  VIN, which a 6.3 V part at 4.5 V does not reliably give.
- C6 becomes 1 uF 16 V, to keep useful capacitance at 4.2 V on the BAT pin.
- R7 at 18 kOhm and R8 at 1.20 kOhm are confirmed correct: table 6-1 gives
  4.2 V and a 500 mA input limit for 18 kOhm, and 300/1200 is 250 mA.
- The bi-colour LED is confirmed safe on 3.3 V through 1 kOhm: both dies are
  AlGaInP at 2.5 V maximum, so the green is not a 3.2 V InGaN part. Whether
  0.8 to 1.3 mA is bright enough through the light pipe is a bench question.

Also adds export_fab.sh for the Gerber, drill, pick-and-place, BOM, assembl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
Parts:
- C6: value 1uF 10V -> 1uF 16V
- C8: value 10uF 6.3V -> 10uF 25V; footprint Capacitor_SMD:C_0603_1608Metric -> Capacitor_SMD:C_0805_2012Metric
Changed lines of the file:
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@@
 			)
 		)
-		(property "Value" "10uF 6.3V"
+		(property "Value" "10uF 25V"
 			(at 167.64 89.916 0)
 			(show_name no)
@@
 			)
 		)
-		(property "Footprint" "Capacitor_SMD:C_0603_1608Metric"
+		(property "Footprint" "Capacitor_SMD:C_0805_2012Metric"
 			(at 175.26 88.9 0)
 			(hide yes)
@@
 			)
 		)
-		(property "Value" "1uF 10V"
+		(property "Value" "1uF 16V"
 			(at 73.914 149.098 0)
 			(show_name no)
