File: hardware/pcb/cicala_rev_a/sheets/battery_charger.kicad_sch (KiCad schematic)
At the start: 35 parts, among them J1 USB-C receptacle, J3 Protected LiPo + NTC, U2 BQ25185DLH, U3 TPS63802DLA, U4 USBLC6-2SC6, U5 TPS22917DBVR

Commit message: feat(hw): finalize Rev A prototype hardware and firmware
Complete the PCB and enclosure review, correct component ratings and footprints, add fitted 3D models, and export validated fabrication, assembly and print files.

Add Rev A firmware configuration, charger and power handling, USB flash/debug support, integration coverage, and build and manufacturing instructions.

Validation: zero configured ERC/DRC/parity findings; 45 PCB/export and 6 mesh tests; 14 nominal fit checks; 226 firmware cases passed with 3 platform skips; debug, charset and release/MCUboot builds; 84 Python and 101 website tests; strict docs build; prototype archive CRC/SHA256 verification. Physical prototype acceptance and factory CAM review remain pending.
Parts:
- added C34: 10uF 10V, Capacitor_SMD:C_0603_1608Metric, symbol Device:C
- C10: value 47uF 6.3V -> 47uF 10V; LCSC (none) -> C41796773; MPN (none) -> CL21A476MPYNNNE; Manufacturer (none) -> Samsung Electro-Mechanics
- C11, C7: LCSC (none) -> C1591; MPN (none) -> CL10B104KB8NNNC; Manufacturer (none) -> Samsung Electro-Mechanics
- C31: value 1nF 2kV -> 1nF 2kV DNP; now not fitted
- C4: value 1uF 25V -> 10uF 10V; LCSC (none) -> C19702; MPN (none) -> CL10A106KP8NNNC; Manufacturer (none) -> Samsung Electro-Mechanics
- C5: LCSC (none) -> C15850; MPN (none) -> CL21A106KAYNNNE; Manufacturer (none) -> Samsung Electro-Mechanics
- C6: value 1uF 16V -> 10uF 10V; LCSC (none) -> C19702; MPN (none) -> CL10A106KP8NNNC; Manufacturer (none) -> Samsung Electro-Mechanics
- C8: value 10uF 25V -> 47uF 10V; LCSC (none) -> C41796773; MPN (none) -> CL21A476MPYNNNE; Manufacturer (none) -> Samsung Electro-Mechanics
- C9: LCSC (none) -> C59461; MPN (none) -> CL10A226MQ8NRNC; Manufacturer (none) -> Samsung Electro-Mechanics
- J1: Manufacturer (none) -> HRO
- J3: MPN custom 503035 pack harness -> S3B-PH-SM4-TB(LF)(SN); Manufacturer (none) -> JST
- L2: Manufacturer (none) -> Coilcraft
- R1, R2: MPN (none) -> RC0603FR-075K1L; Manufacturer (none) -> Yageo
- R10, R9: MPN (none) -> RC0603FR-0710KL; Manufacturer (none) -> Yageo
- R11: MPN (none) -> RC0603FR-071ML; Manufacturer (none) -> Yageo
- R12: MPN (none) -> RC0603FR-07470KL; Manufacturer (none) -> Yageo
- R13: value 100k -> 4.7k; MPN (none) -> RC0603FR-074K7L; Manufacturer (none) -> Yageo
- R14: MPN (none) -> RC0603FR-07511KL; Manufacturer (none) -> Yageo
- R15: MPN (none) -> RC0603FR-0791KL; Manufacturer (none) -> Yageo
- R16: MPN (none) -> RC0603FR-07100KL; Manufacturer (none) -> Yageo
- R3, R4: MPN (none) -> RC0603FR-0722RL; Manufacturer (none) -> Yageo
- R33, R34: MPN (none) -> RC0603JR-070RL; Manufacturer (none) -> Yageo
- R7: MPN (none) -> RC0603FR-0718KL; Manufacturer (none) -> Yageo
- R8: MPN (none) -> RC0603FR-071K2L; Manufacturer (none) -> Yageo
- U2, U3, U5: Manufacturer (none) -> Texas Instruments
- U4: Manufacturer (none) -> STMicroelectronics
Connections:
- net CHG_ENABLE: no longer U2.4 (~{CE})
- net GND: now also C34.2
- net VBAT: now also C34.1
- new net CHG_CE: U2.4 (~{CE})
