File: hardware/pcb/cicala_rev_a/sheets/epaper.kicad_sch (KiCad schematic)
At the start: 23 parts, among them J2 FH12-24S-0.5SH, Q1 Si1308EDL, U6 TPS22917DBVR

Commit message: feat: rename project and adopt Cicala identity
Parts:
- L1: footprint kveld:L_TDK_VLS4012 -> cicala:L_TDK_VLS4012
Changed lines of the file:
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@@
 		)
 		(instances
-			(project "kveld_rev_a"
+			(project "cicala_rev_a"
 				(path "/9b5e4c31-c66f-4b64-9ff8-62a2c447d0bc/9467d62a-f8ed-46c9-a7cb-f7af887ddb15"
 					(reference "#PWR0155")
@@
 		)
 		(instances
-			(project "kveld_rev_a"
+			(project "cicala_rev_a"
 				(path "/9b5e4c31-c66f-4b64-9ff8-62a2c447d0bc/9467d62a-f8ed-46c9-a7cb-f7af887ddb15"
 					(reference "#PWR0145")
@@
 		)
 		(instances
-			(project "kveld_rev_a"
+			(project "cicala_rev_a"
 				(path "/9b5e4c31-c66f-4b64-9ff8-62a2c447d0bc/9467d62a-f8ed-46c9-a7cb-f7af887ddb15"
 					(reference "Q1")
@@
 		)
 		(instances
-			(project "kveld_rev_a"
+			(project "cicala_rev_a"
 				(path "/9b5e4c31-c66f-4b64-9ff8-62a2c447d0bc/9467d62a-f8ed-46c9-a7cb-f7af887ddb15"
 					(reference "C24")
@@
 		)
 		(instances
-			(project "kveld_rev_a"
+			(project "cicala_rev_a"
 				(path "/9b5e4c31-c66f-4b64-9ff8-62a2c447d0bc/9467d62a-f8ed-46c9-a7cb-f7af887ddb15"
 					(reference "C18")
@@
 		)
 		(instances
-			(project "kveld_rev_a"
+			(project "cicala_rev_a"
 				(path "/9b5e4c31-c66f-4b64-9ff8-62a2c447d0bc/9467d62a-f8ed-46c9-a7cb-f7af887ddb15"
 					(reference "C19")
@@
 		)
 		(instances
-			(project "kveld_rev_a"
+			(project "cicala_rev_a"
 				(path "/9b5e4c31-c66f-4b64-9ff8-62a2c447d0bc/9467d62a-f8ed-46c9-a7cb-f7af887ddb15"
 					(reference "#PWR0143")
@@
 		)
 		(instances
-			(project "kveld_rev_a"
+			(project "cicala_rev_a"
 				(path "/9b5e4c31-c66f-4b64-9ff8-62a2c447d0bc/9467d62a-f8ed-46c9-a7cb-f7af887ddb15"
 					(reference "D2")
@@
 		)
 		(instances
-			(project "kveld_rev_a"
+			(project "cicala_rev_a"
 				(path "/9b5e4c31-c66f-4b64-9ff8-62a2c447d0bc/9467d62a-f8ed-46c9-a7cb-f7af887ddb15"
 					(reference "#PWR0144")
@@
 		)
 		(instances
-			(project "kveld_rev_a"
+			(project "cicala_rev_a"
 				(path "/9b5e4c31-c66f-4b64-9ff8-62a2c447d0bc/9467d62a-f8ed-46c9-a7cb-f7af887ddb15"
 					(reference "D3")
@@
 		)
 		(instances
-			(project "kveld_rev_a"
+			(project "cicala_rev_a"
 				(path "/9b5e4c31-c66f-4b64-9ff8-62a2c447d0bc/9467d62a-f8ed-46c9-a7cb-f7af887ddb15"
 					(reference "#PWR0148")
@@
 		)
 		(instances
-			(project "kveld_rev_a"
+			(project "cicala_rev_a"
 				(path "/9b5e4c31-c66f-4b64-9ff8-62a2c447d0bc/9467d62a-f8ed-46c9-a7cb-f7af887ddb15"
 					(reference "#PWR0149")
@@
 		)
 		(instances
-			(project "kveld_rev_a"
+			(project "cicala_rev_a"
 				(path "/9b5e4c31-c66f-4b64-9ff8-62a2c447d0bc/9467d62a-f8ed-46c9-a7cb-f7af887ddb15"
 					(reference "C13")
@@
 		)
 		(instances
-			(project "kveld_rev_a"
+			(project "cicala_rev_a"
 				(path "/9b5e4c31-c66f-4b64-9ff8-62a2c447d0bc/9467d62a-f8ed-46c9-a7cb-f7af887ddb15"
 					(reference "R20")
@@
 		)
 		(instances
-			(project "kveld_rev_a"
+			(project "cicala_rev_a"
 				(path "/9b5e4c31-c66f-4b64-9ff8-62a2c447d0bc/9467d62a-f8ed-46c9-a7cb-f7af887ddb15"
 					(reference "#PWR0146")
@@
 		)
 		(instances
-			(project "kveld_rev_a"
+			(project "cicala_rev_a"
 				(path "/9b5e4c31-c66f-4b64-9ff8-62a2c447d0bc/9467d62a-f8ed-46c9-a7cb-f7af887ddb15"
 					(reference "C22")
@@
 		)
 		(instances
-			(project "kveld_rev_a"
+			(project "cicala_rev_a"
 				(path "/9b5e4c31-c66f-4b64-9ff8-62a2c447d0bc/9467d62a-f8ed-46c9-a7cb-f7af887ddb15"
 					(reference "C21")
@@
 		)
 		(instances
-			(project "kveld_rev_a"
+			(project "cicala_rev_a"
 				(path "/9b5e4c31-c66f-4b64-9ff8-62a2c447d0bc/9467d62a-f8ed-46c9-a7cb-f7af887ddb15"
 					(reference "C20")
@@
 		)
 		(instances
-			(project "kveld_rev_a"
+			(project "cicala_rev_a"
 				(path "/9b5e4c31-c66f-4b64-9ff8-62a2c447d0bc/9467d62a-f8ed-46c9-a7cb-f7af887ddb15"
 					(reference "C15")
@@
 		)
 		(instances
-			(project "kveld_rev_a"
+			(project "cicala_rev_a"
 				(path "/9b5e4c31-c66f-4b64-9ff8-62a2c447d0bc/9467d62a-f8ed-46c9-a7cb-f7af887ddb15"
 					(reference "D1")
@@
 		)
 		(instances
-			(project "kveld_rev_a"
+			(project "cicala_rev_a"
 				(path "/9b5e4c31-c66f-4b64-9ff8-62a2c447d0bc/9467d62a-f8ed-46c9-a7cb-f7af887ddb15"
 					(reference "#PWR0150")
@@
 		)
 		(instances
-			(project "kveld_rev_a"
+			(project "cicala_rev_a"
 				(path "/9b5e4c31-c66f-4b64-9ff8-62a2c447d0bc/9467d62a-f8ed-46c9-a7cb-f7af887ddb15"
 					(reference "C23")
@@
 		)
 		(instances
-			(project "kveld_rev_a"
+			(project "cicala_rev_a"
 				(path "/9b5e4c31-c66f-4b64-9ff8-62a2c447d0bc/9467d62a-f8ed-46c9-a7cb-f7af887ddb15"
 					(reference "C16")
@@
 		)
 		(instances
-			(project "kveld_rev_a"
+			(project "cicala_rev_a"
 				(path "/9b5e4c31-c66f-4b64-9ff8-62a2c447d0bc/9467d62a-f8ed-46c9-a7cb-f7af887ddb15"
 					(reference "#PWR0142")
@@
 		)
 		(instances
-			(project "kveld_rev_a"
+			(project "cicala_rev_a"
 				(path "/9b5e4c31-c66f-4b64-9ff8-62a2c447d0bc/9467d62a-f8ed-46c9-a7cb-f7af887ddb15"
 					(reference "J2")
@@
 		)
 		(instances
-			(project "kveld_rev_a"
+			(project "cicala_rev_a"
 				(path "/9b5e4c31-c66f-4b64-9ff8-62a2c447d0bc/9467d62a-f8ed-46c9-a7cb-f7af887ddb15"
 					(reference "#PWR0154")
@@
 		)
 		(instances
-			(project "kveld_rev_a"
+			(project "cicala_rev_a"
 				(path "/9b5e4c31-c66f-4b64-9ff8-62a2c447d0bc/9467d62a-f8ed-46c9-a7cb-f7af887ddb15"
 					(reference "U6")
@@
 		)
 		(instances
-			(project "kveld_rev_a"
+			(project "cicala_rev_a"
 				(path "/9b5e4c31-c66f-4b64-9ff8-62a2c447d0bc/9467d62a-f8ed-46c9-a7cb-f7af887ddb15"
 					(reference "C12")
@@
 		)
 		(instances
-			(project "kveld_rev_a"
+			(project "cicala_rev_a"
 				(path "/9b5e4c31-c66f-4b64-9ff8-62a2c447d0bc/9467d62a-f8ed-46c9-a7cb-f7af887ddb15"
 					(reference "#PWR0141")
@@
 		)
 		(instances
-			(project "kveld_rev_a"
+			(project "cicala_rev_a"
 				(path "/9b5e4c31-c66f-4b64-9ff8-62a2c447d0bc/9467d62a-f8ed-46c9-a7cb-f7af887ddb15"
 					(reference "R19")
@@
 			)
 		)
-		(property "Footprint" "kveld:L_TDK_VLS4012"
+		(property "Footprint" "cicala:L_TDK_VLS4012"
 			(at 104.14 50.8 0)
 			(hide yes)
@@
 		)
 		(instances
-			(project "kveld_rev_a"
+			(project "cicala_rev_a"
 				(path "/9b5e4c31-c66f-4b64-9ff8-62a2c447d0bc/9467d62a-f8ed-46c9-a7cb-f7af887ddb15"
 					(reference "L1")
@@
 		)
 		(instances
-			(project "kveld_rev_a"
+			(project "cicala_rev_a"
 				(path "/9b5e4c31-c66f-4b64-9ff8-62a2c447d0bc/9467d62a-f8ed-46c9-a7cb-f7af887ddb15"
 					(reference "#PWR0153")
@@
 		)
 		(instances
-			(project "kveld_rev_a"
+			(project "cicala_rev_a"
 				(path "/9b5e4c31-c66f-4b64-9ff8-62a2c447d0bc/9467d62a-f8ed-46c9-a7cb-f7af887ddb15"
 					(reference "C14")
@@
 		)
 		(instances
-			(project "kveld_rev_a"
+			(project "cicala_rev_a"
 				(path "/9b5e4c31-c66f-4b64-9ff8-62a2c447d0bc/9467d62a-f8ed-46c9-a7cb-f7af887ddb15"
 					(reference "#PWR0151")
@@
 		)
 		(instances
-			(project "kveld_rev_a"
+			(project "cicala_rev_a"
 				(path "/9b5e4c31-c66f-4b64-9ff8-62a2c447d0bc/9467d62a-f8ed-46c9-a7cb-f7af887ddb15"
 					(reference "#PWR0152")
@@
 		)
 		(instances
-			(project "kveld_rev_a"
+			(project "cicala_rev_a"
 				(path "/9b5e4c31-c66f-4b64-9ff8-62a2c447d0bc/9467d62a-f8ed-46c9-a7cb-f7af887ddb15"
 					(reference "#PWR0147")
@@
 		)
 		(instances
-			(project "kveld_rev_a"
+			(project "cicala_rev_a"
 				(path "/9b5e4c31-c66f-4b64-9ff8-62a2c447d0bc/9467d62a-f8ed-46c9-a7cb-f7af887ddb15"
 					(reference "R18")
@@
 		)
 		(instances
-			(project "kveld_rev_a"
+			(project "cicala_rev_a"
 				(path "/9b5e4c31-c66f-4b64-9ff8-62a2c447d0bc/9467d62a-f8ed-46c9-a7cb-f7af887ddb15"
 					(reference "C17")
