File: hardware/pcb/cicala_rev_a/sheets/epaper.kicad_sch (KiCad schematic)
At the start: 35 parts, among them J2 GDEY0213B74, Q1 Si1308EDL, U6 TPS22917DBVR

Commit message: refactor(hw): make the root sheet a real hierarchy
The root was three boxes and a filename; every cross-sheet signal travelled
by global label, so nothing recorded which block produced a signal and which
consumed it. The 19 nets that actually cross a sheet boundary are now
hierarchical: each child carries a directional hierarchical label and the
root carries the matching sheet pin, wired block to block. The root also
states the power flow in words.

GND stays global; a ground symbol reads better than a pin on every block.
Root-level global labels keep the plain net names that pin_contract.csv and
the firmware refer to, rather than the sheet-path names a local label gives.

Connectivity is unchanged: the exported netlist is identical to the one
before the conversion, net for net and pin for pin.

Also hides the PWR_FLAG references, moves the USB shield network and the
cell-current link inside the blocks they belong to, and gives every page the
same company, revision and date.

Co-Authored-By: Claude Opus 5 <noreply@anthropic.com>
Claude-Session: https://claude.ai/code/session_01E5vy1HJsPztSk9nFw6j5Ko
Other:
- company: (none) -> Cicala
Changed lines of the file:
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@@
 		(title "GDEY0213B74 e-paper interface and boost")
 		(rev "Rev A")
+		(date "2026-09-05")
+		(company "Cicala")
 	)
 	(rectangle
@@
 		)
 	)
-	(global_label "EPD_BUSY"
-		(shape passive)
+	(hierarchical_label "EPD_BUSY"
+		(shape output)
 		(at 33.02 147.32 0)
 		(fields_autoplaced yes)
@@
 			(justify left)
 		)
-		(property "Intersheetrefs" "${INTERSHEET_REFS}"
-			(at 33.02 147.32 0)
-			(hide yes)
-			(show_name no)
-			(do_not_autoplace no)
-			(effects
-				(font
-					(size 0.8 0.8)
-				)
-			)
-		)
 	)
 	(global_label "EPD_VGL"
@@
 		)
 	)
-	(global_label "3V3"
-		(shape passive)
+	(hierarchical_label "3V3"
+		(shape input)
 		(at 190.5 113.03 90)
 		(fields_autoplaced yes)
@@
 			(justify left)
 		)
-		(property "Intersheetrefs" "${INTERSHEET_REFS}"
-			(at 190.5 113.03 0)
-			(hide yes)
-			(show_name no)
-			(do_not_autoplace no)
-			(effects
-				(font
-					(size 0.8 0.8)
-				)
-			)
-		)
 	)
 	(global_label "EPD_3V3"
@@
 		)
 	)
-	(global_label "3V3"
-		(shape passive)
+	(hierarchical_label "3V3"
+		(shape input)
 		(at 31.75 38.1 180)
 		(fields_autoplaced yes)
@@
 			(justify right)
 		)
-		(property "Intersheetrefs" "${INTERSHEET_REFS}"
-			(at 31.75 38.1 0)
-			(hide yes)
-			(show_name no)
-			(do_not_autoplace no)
-			(effects
-				(font
-					(size 0.8 0.8)
-				)
-			)
-		)
 	)
 	(global_label "EPD_PUMP"
@@
 		)
 	)
-	(global_label "EPD_PWR_EN"
-		(shape passive)
+	(hierarchical_label "EPD_PWR_EN"
+		(shape input)
 		(at 31.75 43.18 180)
 		(fields_autoplaced yes)
@@
 			(justify right)
 		)
-		(property "Intersheetrefs" "${INTERSHEET_REFS}"
-			(at 31.75 43.18 0)
-			(hide yes)
-			(show_name no)
-			(do_not_autoplace no)
-			(effects
-				(font
-					(size 0.8 0.8)
-				)
-			)
-		)
 	)
 	(global_label "PNL_CLK"
@@
 		)
 	)
-	(global_label "3V3"
-		(shape passive)
+	(hierarchical_label "3V3"
+		(shape input)
 		(at 20.32 59.69 270)
 		(fields_autoplaced yes)
@@
 			(justify left)
 		)
-		(property "Intersheetrefs" "${INTERSHEET_REFS}"
-			(at 20.32 59.69 0)
-			(hide yes)
-			(show_name no)
-			(do_not_autoplace no)
-			(effects
-				(font
-					(size 0.8 0.8)
-				)
-			)
-		)
 	)
 	(wire
@@
 		)
 	)
-	(global_label "EPD_CLK"
-		(shape passive)
+	(hierarchical_label "EPD_CLK"
+		(shape input)
 		(at 78.74 127.0 0)
 		(fields_autoplaced yes)
@@
 			(justify left)
 		)
-		(property "Intersheetrefs" "${INTERSHEET_REFS}"
-			(at 78.74 127.0 0)
-			(hide yes)
-			(show_name no)
-			(do_not_autoplace no)
-			(effects
-				(font
-					(size 0.8 0.8)
-				)
-			)
-		)
 	)
 	(global_label "PNL_MOSI"
@@
 		)
 	)
-	(global_label "EPD_MOSI"
-		(shape passive)
+	(hierarchical_label "EPD_MOSI"
+		(shape input)
 		(at 78.74 134.62 0)
 		(fields_autoplaced yes)
@@
 			(justify left)
 		)
-		(property "Intersheetrefs" "${INTERSHEET_REFS}"
-			(at 78.74 134.62 0)
-			(hide yes)
-			(show_name no)
-			(do_not_autoplace no)
-			(effects
-				(font
-					(size 0.8 0.8)
-				)
-			)
-		)
 	)
 	(global_label "PNL_CS"
@@
 		)
 	)
-	(global_label "EPD_CS"
-		(shape passive)
+	(hierarchical_label "EPD_CS"
+		(shape input)
 		(at 78.74 142.24 0)
 		(fields_autoplaced yes)
@@
 			(justify left)
 		)
-		(property "Intersheetrefs" "${INTERSHEET_REFS}"
-			(at 78.74 142.24 0)
-			(hide yes)
-			(show_name no)
-			(do_not_autoplace no)
-			(effects
-				(font
-					(size 0.8 0.8)
-				)
-			)
-		)
 	)
 	(global_label "PNL_DC"
@@
 		)
 	)
-	(global_label "EPD_DC"
-		(shape passive)
+	(hierarchical_label "EPD_DC"
+		(shape input)
 		(at 78.74 149.86 0)
 		(fields_autoplaced yes)
@@
 			(justify left)
 		)
-		(property "Intersheetrefs" "${INTERSHEET_REFS}"
-			(at 78.74 149.86 0)
-			(hide yes)
-			(show_name no)
-			(do_not_autoplace no)
-			(effects
-				(font
-					(size 0.8 0.8)
-				)
-			)
-		)
 	)
 	(global_label "PNL_RESET"
@@
 		)
 	)
-	(global_label "EPD_RESET"
-		(shape passive)
+	(hierarchical_label "EPD_RESET"
+		(shape input)
 		(at 78.74 157.48 0)
 		(fields_autoplaced yes)
@@
 			(justify left)
 		)
-		(property "Intersheetrefs" "${INTERSHEET_REFS}"
-			(at 78.74 157.48 0)
-			(hide yes)
-			(show_name no)
-			(do_not_autoplace no)
-			(effects
-				(font
-					(size 0.8 0.8)
-				)
-			)
-		)
 	)
 	(junction
@@
 		)
 	)
-	(global_label "EPD_BUSY"
-		(shape passive)
+	(hierarchical_label "EPD_BUSY"
+		(shape output)
 		(at 162.56 160.02 270)
 		(fields_autoplaced yes)
@@
 			(justify left)
 		)
-		(property "Intersheetrefs" "${INTERSHEET_REFS}"
-			(at 162.56 160.02 0)
-			(hide yes)
-			(show_name no)
-			(do_not_autoplace no)
-			(effects
-				(font
-					(size 0.8 0.8)
-				)
-			)
-		)
 	)
