File: hardware/pcb/cicala_rev_a/sheets/epaper.kicad_sch (KiCad schematic)
At the start: 35 parts, among them J2 GDEY0213B74, Q1 Si1308EDL, U6 TPS22917DBVR

Commit message: feat(hw): finalize Rev A prototype hardware and firmware
Complete the PCB and enclosure review, correct component ratings and footprints, add fitted 3D models, and export validated fabrication, assembly and print files.

Add Rev A firmware configuration, charger and power handling, USB flash/debug support, integration coverage, and build and manufacturing instructions.

Validation: zero configured ERC/DRC/parity findings; 45 PCB/export and 6 mesh tests; 14 nominal fit checks; 226 firmware cases passed with 3 platform skips; debug, charset and release/MCUboot builds; 84 Python and 101 website tests; strict docs build; prototype archive CRC/SHA256 verification. Physical prototype acceptance and factory CAM review remain pending.
Parts:
- C12, C17, C18, C19, C20, C21, C22, C23, C24: LCSC (none) -> C29936; MPN (none) -> CL10B105KA8NNNC; Manufacturer (none) -> Samsung Electro-Mechanics
- C13: LCSC (none) -> C19702; MPN (none) -> CL10A106KP8NNNC; Manufacturer (none) -> Samsung Electro-Mechanics
- C14: LCSC (none) -> C163508; MPN (none) -> CL10C102JB8NNNC; Manufacturer (none) -> Samsung Electro-Mechanics
- C15, C16: LCSC (none) -> C98195; MPN (none) -> CL21B475KAFNNNE; Manufacturer (none) -> Samsung Electro-Mechanics
- D1, D2, D3: MPN MBR0530 -> MBR0530-7-F; Manufacturer (none) -> Diodes Incorporated
- J2: Manufacturer (none) -> Hirose
- L1: Manufacturer (none) -> TDK
- Q1: Manufacturer (none) -> Vishay
- R18: MPN (none) -> RC0603FR-07150RL; Manufacturer (none) -> Yageo
- R19, R32: MPN (none) -> RC0603FR-071ML; Manufacturer (none) -> Yageo
- R20: MPN (none) -> RC0603FR-072R2L; Manufacturer (none) -> Yageo
- R27, R28, R29, R30, R31: MPN (none) -> RC0603FR-07470RL; Manufacturer (none) -> Yageo
- U6: Manufacturer (none) -> Texas Instruments
Other:
- moved on the sheet: C16, D1, D2, J2, R27, R28, R29, R30, R31, R32, TP16, TP17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
