File: hardware/pcb/cicala_rev_a/sheets/esp32_core.kicad_sch (KiCad schematic)
At the start: 35 parts, among them J4 TC2030 recovery pads, SW1 CATEGORY KSC321GLFS, SW2 NEXT KSC321GLFS, U1 ESP32-S3-WROOM-1-N16 / WROOM-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

Commit message: feat(hw): finalize Rev A prototype hardware and firmware
Complete the PCB and enclosure review, correct component ratings and footprints, add fitted 3D models, and export validated fabrication, assembly and print files.

Add Rev A firmware configuration, charger and power handling, USB flash/debug support, integration coverage, and build and manufacturing instructions.

Validation: zero configured ERC/DRC/parity findings; 45 PCB/export and 6 mesh tests; 14 nominal fit checks; 226 firmware cases passed with 3 platform skips; debug, charset and release/MCUboot builds; 84 Python and 101 website tests; strict docs build; prototype archive CRC/SHA256 verification. Physical prototype acceptance and factory CAM review remain pending.
Parts:
- C25, C26: LCSC (none) -> C1589; MPN (none) -> CL10B103KB8NNNC; Manufacturer (none) -> Samsung Electro-Mechanics
- C27: LCSC (none) -> C29936; MPN (none) -> CL10B105KA8NNNC; Manufacturer (none) -> Samsung Electro-Mechanics
- C28, C3: LCSC (none) -> C1591; MPN (none) -> CL10B104KB8NNNC; Manufacturer (none) -> Samsung Electro-Mechanics
- C29: LCSC (none) -> C19702; MPN (none) -> CL10A106KP8NNNC; Manufacturer (none) -> Samsung Electro-Mechanics
- C30: value 47uF -> 47uF 10V; LCSC (none) -> C41796773; MPN (none) -> CL21A476MPYNNNE; Manufacturer (none) -> Samsung Electro-Mechanics
- D4: symbol Device:LED_Dual_AAKK -> Cicala:APBA2006SURKCGKC; Manufacturer (none) -> Kingbright
- J4: now fitted
- R21, R22: value 47k -> 22k; MPN (none) -> RC0603FR-0722KL; Manufacturer (none) -> Yageo
- R23, R24: MPN (none) -> RC0603FR-071KL; Manufacturer (none) -> Yageo
- R25, R26: MPN (none) -> RC0603FR-0710KL; Manufacturer (none) -> Yageo
- R5: MPN (none) -> RC0603FR-07100KL; Manufacturer (none) -> Yageo
- R6: MPN (none) -> RC0603FR-07150KL; Manufacturer (none) -> Yageo
- SW1: value CATEGORY KSC321GLFS -> CATEGORY KSC323GLFG; MPN KSC321GLFS -> KSC323GLFG; Manufacturer (none) -> C&K
- SW2: value NEXT KSC321GLFS -> NEXT KSC323GLFG; MPN KSC321GLFS -> KSC323GLFG; Manufacturer (none) -> C&K
- U1: value ESP32-S3-WROOM-1-N16 / WROOM-1U-N16 -> ESP32-S3-WROOM-1-N16; MPN ESP32-S3-WROOM-1-N16; alt ESP32-S3-WROOM-1U-N16 -> ESP32-S3-WROOM-1-N16; Manufacturer (none) -> Espressif Systems
Other:
- note added: "Module decoupling"
- moved on the sheet: C28, C29, C30, TP1, TP10, TP11, TP12, TP13, TP14, TP15, TP2, TP3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
