File: hardware/rev_b/pcb/cicala_rev_b.kicad_pcb (KiCad board)
At the start: 4 copper layers, 103 x 62 mm, 115 parts, among them J1 USB-C receptacle, J2 Waveshare 3.52in V1.1 UC8253, J3 Battery + external 10k B3435 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, J4 TC2030 recovery pads, Q1 BSS138, Q2 2N7002P, SW1 SKRABCE010, SW2 SKRABCE010, U1 ESP32-S3-WROOM-1-N16, U2 BQ25185DLH, U3 TPS63802DLA, U4 USBLC6-2SC6, U5 TPS22917DBVR, U6 TPS22917DBVR, U7 TLV9022DGK

Commit message: feat(hw): add board legends and straight PCB views
Other:
- board text added: "+"
- board text added: "-"
- board text added: "01 DISPLAY / BOOST"
- board text added: "02 NTC GUARD"
- board text added: "03 POWER"
- board text added: "1 3V3 2 GND 3 EN"
- board text added: "1 BOOT 2 EN 3 GND"
- board text added: "10 5V 14 STAT1"
- board text added: "100mA"
- board text added: "11 PGOOD"
- board text added: "15 STAT2"
- board text added: "16 CLK 17 MOSI"
- board text added: "18 CS 19 DC 21 BUSY"
- board text added: "20 RESET"
- board text added: "22 CELL+"
- board text added: "3V3"
- board text added: "3V3 REF ONLY / NO POWER"
- board text added: "4 BOOT 5 TX 6 RX"
- board text added: "4 LAYERS / 1.2mm / PROTOTYPE"
- board text added: "4 TX"
- board text added: "5 RX"
- board text added: "5V"
- board text added: "6 FACTORY OD"
- board text added: "7 3V3 8 BAT 9 SYS"
- board text added: "ANTENNA / KEEP CLEAR"
- board text added: "B.03"
- board text added: "BAT"
- board text added: "BOOT"
- board text added: "BOOT LOW + PULSE EN"
- board text added: "BUSY"
- board text added: "CERN-OHL-S-2.0"
- board text added: "CLK"
- board text added: "CONTACTS DOWN"
- board text added: "CS"
- board text added: "D4 STATUS"
- board text added: "DC"
- board text added: "DEBUG"
- board text added: "EN"
- board text added: "GND"
- board text added: "J2 E-PAPER"
- board text added: "J2 UC8253 / CONTACTS DOWN"
- board text added: "J3 1:+ 2:NTC 3:GND"
- board text added: "J3 BAT"
- board text added: "J4"
- board text added: "J4 RECOVERY / 3V3 LOGIC"
- board text added: "L1"
- board text added: "LiPo <-> U2 / VSYS -> U3 -> 3V3"
- board text added: "MOSI"
- board text added: "NTC 10k B3435 ON CELL"
- board text added: "POWER: USB 5V -> U2 -> VSYS"
- board text added: "PROTECTED 1S LiPo ONLY"
- board text added: "REV B.03 / ESP32-S3 / 16MB"
- board text added: "REV B.03 ENGINEERING PROTOTYPE - PHYSICAL QUALIFICATION PENDING"
- board text added: "S1"
- board text added: "SW1 FILTERS"
- board text added: "SW2 NEXT"
- board text added: "SYS"
- board text added: "T"
- board text added: "TOP TEST POINTS"
- board text added: "TX / RX FROM MCU"
- board text added: "U1 ESP32-S3 / 16MB"
- board text added: "U2 BQ25185: 100mA CHARGE"
- board text added: "U2 CHARGE"
- board text added: "U3 3V3"
- board text added: "U6"
- board text added: "U7"
- board text added: "U7 + Q2: NTC CHARGE GUARD"
- board text added: "USB 5V / DATA"
- board text removed: "REV B FIT ONLY - UNROUTED - DO NOT FABRICATE"

Commit message: feat(hw): simplify Rev B controls with purchased Omron caps
Parts:
- SW1, SW2: value SKRABCE010 -> B3F-4050; footprint cicala:SW_Alps_SKRABCE010 -> cicala:SW_Omron_B3F-4050
- moved SW1 5.40 mm to (108.0, 17.5), turned to 0 degrees
- moved SW2 5.40 mm to (108.0, 52.3), turned to 0 degrees
Routing:
- net BTN_CATEGORY: track 115.2 -> 131.4 mm
- net BTN_NEXT: track 110.5 -> 124.9 mm
- net GND: track 83.4 -> 79.9 mm, vias 154 -> 149
Other:
- board size 103 x 62 mm -> 113 x 62 mm
- board text added: "B.04"
- board text added: "REV B.04 / ESP32-S3 / 16MB"
- board text added: "REV B.04 ENGINEERING PROTOTYPE - PHYSICAL QUALIFICATION PENDING"
- board text removed: "B.03"
- board text removed: "REV B.03 / ESP32-S3 / 16MB"
- board text removed: "REV B.03 ENGINEERING PROTOTYPE - PHYSICAL QUALIFICATION PENDING"

Commit message: fix(hw): recess Rev B controls and prepare first-article files
Routing:
- net GND: track 79.9 -> 76.3 mm, vias 149 -> 147
- net BTN_NEXT: track 124.9 -> 122.7 mm
Other:
- board text added: "B.05"
- board text added: "REV B.05 / ESP32-S3 / 16MB"
- board text added: "REV B.05 ENGINEERING PROTOTYPE - PHYSICAL QUALIFICATION PENDING"
- board text removed: "B.04"
- board text removed: "REV B.04 / ESP32-S3 / 16MB"
- board text removed: "REV B.04 ENGINEERING PROTOTYPE - PHYSICAL QUALIFICATION PENDING"
