File: hardware/rev_b/pcb/cicala_rev_b.kicad_sch (KiCad schematic)
At the start: 0 parts

Commit message: fix(hw): recess Rev B controls and prepare first-article files
Other:
- note added: "Cicala Rev B.05 system block diagram"
- note removed: "Cicala Rev B FIT STUDY system block diagram"
- note removed: "UNROUTED FIT STUDY — no firmware target / no fabrication release"
- title: Cicala Rev B FIT STUDY schematic overview -> Cicala Rev B.05 schematic overview
Changed lines of the file:
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@@
 	(paper "A4")
 	(title_block
-		(title "Cicala Rev B FIT STUDY schematic overview")
-		(date "2026-09-07")
-		(rev "Rev B FIT - NOT FOR FABRICATION")
+		(title "Cicala Rev B.05 schematic overview")
+		(date "2026-09-16")
+		(rev "B.05")
 		(company "Cicala")
+		(comment 1 "Engineering prototype; physical qualification pending")
 	)
 	(text "Power flow: USB-C 5 V or the protected cell -> BQ25185 power path (VSYS)\n-> TPS63802 buck-boost (3V3) -> TPS22917 load switches, one for the\nbattery divider and one for the panel and its boost network."
@@
 		)
 	)
-	(text "Cicala Rev B FIT STUDY system block diagram"
+	(text "Cicala Rev B.05 system block diagram"
 		(exclude_from_sim no)
 		(at 20.32 25.4 0)
@@
 		)
 	)
-	(text "UNROUTED FIT STUDY — no firmware target / no fabrication release"
-		(at 20 185 0)
-		(effects
-			(font
-				(size 1.27 1.27)
-			)
-			(justify left)
-		)
-	)
