File: hardware/rev_b/pcb/sheets/battery_charger.kicad_sch (KiCad schematic)
At the start: 34 parts, among them J1 USB-C receptacle, J3 Battery + external 10k B3435 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, U2 BQ25185DLH, U3 TPS63802DLA, U4 USBLC6-2SC6, U5 TPS22917DBVR

Commit message: fix(hw): recess Rev B controls and prepare first-article files
Other:
- note removed: "UNROUTED FIT STUDY — no firmware target / no fabrication release"
Changed lines of the file:
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@@
 	(title_block
 		(title "Power, charging, and USB")
-		(date "2026-09-07")
-		(rev "Rev B FIT - NOT FOR FABRICATION")
+		(date "2026-09-16")
+		(rev "B.05")
 		(company "Cicala")
+		(comment 1 "Engineering prototype; physical qualification pending")
 	)
 	(rectangle
@@
 		)
 	)
-	(text "UNROUTED FIT STUDY — no firmware target / no fabrication release"
-		(at 20 185 0)
-		(effects
-			(font
-				(size 1.27 1.27)
-			)
-			(justify left)
-		)
-	)
