File: hardware/rev_b/pcb/sheets/epaper.kicad_sch (KiCad schematic)
At the start: 35 parts, among them J2 Waveshare 3.52in V1.1 UC8253, Q1 BSS138, U6 TPS22917DBVR

Commit message: fix(hw): recess Rev B controls and prepare first-article files
Other:
- note added: "Panel pinout follows V1.1 table: 1/4 NC, 5 VDHR. Confirm panel revision and rails at first bring-up."
- note removed: "PANEL GATE: V1.1 p5 pin table conflicts with p16 circuit (pins 1/4/5). Boost values unqualified."
- title: Waveshare_352_V11_UC8253 e-paper interface and boost -> UC8253 e-paper interface and boost
Changed lines of the file:
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@@
 	(paper "A4")
 	(title_block
-		(title "Waveshare_352_V11_UC8253 e-paper interface and boost")
-		(date "2026-09-07")
-		(rev "Rev B FIT - NOT FOR FABRICATION")
+		(title "UC8253 e-paper interface and boost")
+		(date "2026-09-16")
+		(rev "B.05")
 		(company "Cicala")
+		(comment 1 "Engineering prototype; physical qualification pending")
 	)
 	(rectangle
@@
 		)
 	)
-	(text "PANEL GATE: V1.1 p5 pin table conflicts with p16 circuit (pins 1/4/5). Boost values unqualified."
-		(at 20 185 0)
+	(text "Panel pinout follows V1.1 table: 1/4 NC, 5 VDHR.\nConfirm panel revision and rails at first bring-up."
+		(at 190 22 0)
 		(effects
 			(font
